Commit message: Add files via upload
update version with extremely better performance

File: bicycle_ros/urdf/bicycle.xacro (robot description, xacro)
@@ -20,6 +20,8 @@
   <link name="back_wheel_1">
     <inertial>
-      <origin xyz="-4.665051260843711e-07 0.07999999999999871 -9.474190248992542e-08" rpy="0 0 0"/>
-      <mass value="8"/>
+      <!--origin xyz="-4.665051260843711e-07 0.07999999999999871 -9.474190248992542e-08" rpy="0 0 0"/-->
+      <origin xyz="0.0 0.08 0.0" rpy="0 0 0"/>
+      <!--mass value="8"/-->
+      <mass value="10"/>
       <inertia ixx="0.226393" iyy="0.449891" izz="0.226393" ixy="-0.0" iyz="0.0" ixz="0.0"/>
     </inertial>
@@ -40,6 +42,8 @@
   <link name="frame">
     <inertial>
-      <origin xyz="-0.4180874824874772 -1.8521219476316816e-08 0.004402431246678269" rpy="0 0 0"/>
-      <mass value="22"/>
+      <!--origin xyz="-0.4180874824874772 -1.8521219476316816e-08 0.004402431246678269" rpy="0 0 0"/-->
+      <origin xyz="-0.4 0 0.0" rpy="0 0 0"/>
+      <!--mass value="22"/-->
+      <mass value="20"/>
       <inertia ixx="0.126115" iyy="0.297787" izz="0.179524" ixy="0.0" iyz="-0.0" ixz="-0.045126"/>
     </inertial>
@@ -60,5 +64,6 @@
   <link name="front_wheel_1">
     <inertial>
-      <origin xyz="-3.1036681114038345e-08 0.08399999999999737 -9.474189649472109e-08" rpy="0 0 0"/>
+      <!--origin xyz="-3.1036681114038345e-08 0.08399999999999737 -9.474189649472109e-08" rpy="0 0 0"/-->
+      <origin xyz="0 0.084 0" rpy="0 0 0"/>
       <mass value="2"/>
       <inertia ixx="0.206376" iyy="0.410961" izz="0.206376" ixy="-0.0" iyz="0.0" ixz="-0.0"/>
@@ -80,5 +85,6 @@
   <link name="front_fork_1">
     <inertial>
-      <origin xyz="0.09904830883535634 -6.450152857772817e-14 -0.20717436570824999" rpy="0 0 0"/>
+      <!--origin xyz="0.09904830883535634 -6.450152857772817e-14 -0.20717436570824999" rpy="0 0 0"/-->
+      <origin xyz="0 0.0 -0.2" rpy="0 0 0"/>
       <mass value="4"/>
       <inertia ixx="0.053195" iyy="0.047325" izz="0.015452" ixy="-0.0" iyz="-0.0" ixz="0.012899"/>
@@ -109,5 +115,5 @@
     <child link="front_wheel_1"/>
     <dynamics damping="0.0" friction="0.0"/>
-    <axis xyz="0.0 -1.0 0.0"/>
+    <axis xyz="0.0 1.0 0.0"/>
   </joint>
   <joint name="Rev3" type="continuous">
