Commit message: graduate version

File: bicycle_ros/urdf/gazebo.xacro (robot description, xacro)
@@ -1,3 +1,4 @@
 <?xml version="1.0" ?>
+<!-- Publishes the ground truth position from Gazebo -->
 <robot name="bicycle" xmlns:xacro="http://www.ros.org/wiki/xacro" >
   <gazebo>

File: bicycle_ros/urdf/obstacle.xacro (robot description, xacro)
@@ -11,5 +11,5 @@
     <origin xyz="0 0 0"/>
     <geometry>
-      <cylinder radius="0.7" length="1.0" />
+      <cylinder radius="0.35" length="1.0" />
     </geometry>
   </visual>
@@ -17,5 +17,6 @@
     <origin xyz="0 0 0"/>
     <geometry>
-      <cylinder radius="0.7" length="1.0" />
+<!--      <cylinder radius="0.7" length="1.0" />-->
+      <cylinder radius="0.3" length="1.0" />
     </geometry>
   </collision>
